Commit message: update the gait_ground

File: robot/urdf/robot.urdf (robot description, URDF)
Before this commit: robot C:\Users\David\desktop\v1_urdf, 23 links, 22 joints
Links:
- link bearing: geometry collision mesh filename=package://assets\merged\bearing_collision.stl; visual mesh filename=package://assets\merged\bearing_visual.stl
- link bicep: geometry collision mesh filename=package://assets\merged\bicep_collision.stl; visual mesh filename=package://assets\merged\bicep_visual.stl
- link camera_enclosure: geometry collision mesh filename=package://assets\merged\camera_enclosure_collision.stl; visual mesh filename=package://assets\merged\camera_enclosure_visual.stl
- link foot: geometry collision mesh filename=package://assets\merged\foot_collision.stl; visual mesh filename=package://assets\merged\foot_visual.stl
- link foot_2: geometry collision mesh filename=package://assets\merged\foot_2_collision.stl; visual mesh filename=package://assets\merged\foot_2_visual.stl
- link forearm: geometry collision mesh filename=package://assets\merged\forearm_collision.stl; visual mesh filename=package://assets\merged\forearm_visual.stl
- link knee_ankle_rotor_case: geometry collision mesh filename=package://assets\merged\knee_ankle_rotor_case_collision.stl; visual mesh filename=package://assets\merged\knee_ankle_rotor_case_visual.stl
- link knee_ankle_rotor_case_2: geometry collision mesh filename=package://assets\merged\knee_ankle_rotor_case_2_collision.s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; visual mesh filename=package://assets\merged\knee_ankle_rotor_case_2_visual.stl
- link knee_housing: geometry collision mesh filename=package://assets\merged\knee_housing_collision.stl; visual mesh filename=package://assets\merged\knee_housing_visual.stl
- link pitch_roll_housing: geometry collision mesh filename=package://assets\merged\pitch_roll_housing_collision.stl; visual mesh filename=package://assets\merged\pitch_roll_housing_visual.stl
- link shoulder_rightangle: geometry collision mesh filename=package://assets\merged\shoulder_rightangle_collision.stl; visual mesh filename=package://assets\merged\shoulder_rightangle_visual.stl
- link shoulder_rightangle_2: geometry collision mesh filename=package://assets\merged\shoulder_rightangle_2_collision.stl; visual mesh filename=package://assets\merged\shoulder_rightangle_2_visual.stl
- link sts3250: geometry collision mesh filename=package://assets\merged\sts3250_collision.stl; visual mesh filename=package://assets\merged\sts3250_visual.stl
- link sts3250_2: geometry collision mesh filename=package://assets\merged\sts3250_2_collision.stl; visual mesh filename=package://assets\merged\sts3250_2_visual.stl
- link sts3250_3: geometry collision mesh filename=package://assets\merged\sts3250_3_collision.stl; visual mesh filename=package://assets\merged\sts3250_3_visual.stl
- link sts3250_4: geometry collision mesh filename=package://assets\merged\sts3250_4_collision.stl; visual mesh filename=package://assets\merged\sts3250_4_visual.stl
- link sts3250_5: geometry collision mesh filename=package://assets\merged\sts3250_5_collision.stl; visual mesh filename=package://assets\merged\sts3250_5_visual.stl
- link sts3250_6: geometry collision mesh filename=package://assets\merged\sts3250_6_collision.stl; visual mesh filename=package://assets\merged\sts3250_6_visual.stl
- link torso: geometry collision mesh filename=package://assets\merged\torso_collision.stl; visual mesh filename=package://assets\merged\torso_visual.stl
- link yaw_adapter: geometry collision mesh filename=package://assets\merged\yaw_adapter_collision.stl; visual mesh filename=package://assets\merged\yaw_adapter_visual.stl
- link yaw_adapter_2: geometry collision mesh filename=package://assets\merged\yaw_adapter_2_collision.stl; visual mesh filename=package://assets\merged\yaw_adapter_2_visual.stl
Joints:
- joint left_sole_joint_fixed: origin xyz=0 0.027 -0.0275 rpy=1.57079632679 0 0 -> xyz=0 0.027 -0.0275 rpy=1.57079632679 1.57079632679 0
- joint right_sole_joint_fixed: origin xyz=0 0.027 -0.0275 rpy=1.57079632679 0 0 -> xyz=0 0.027 -0.0275 rpy=1.57079632679 1.57079632679 0
