Commit message: Completed the robot moves in a straight line along the y-axis.

File: robot/urdf/robot_mod.urdf (robot description, URDF)
Before this commit: robot C:\Users\David\desktop\v1_urdf, 28 links, 27 joints
Links:
- removed link base_link
- removed link pelvis
Joints:
- removed joint base_link_fixed
- removed joint pelvis_fixed
